File: MagneticSensor/MagneticSensor.kicad_pcb (KiCad board)
At the start: 2 copper layers, 32 x 32 mm, 10 parts, among them J1 Conn_01x07_MountingPin, U1 AS5048A

Commit message: Initial mag encoder board
Parts:
- removed TP1, TP2, TP3, TP4, TP5: TestPoint, TestPoint:TestPoint_Pad_D1.0mm
- added C1: 100nf, Capacitor_SMD:C_0402_1005Metric, F.Cu at (150.0, 105.0)
- added C2: 10uf, Capacitor_SMD:C_0603_1608Metric, B.Cu at (162.5, 102.0)
- added D1: LED, LED_SMD:LED_0603_1608Metric, B.Cu at (164.0, 99.0)
- added G***: LOGO, Logo:Logo, F.Cu at (150.0, 110.5)
- added G***: LOGO, Logo:Logo, B.Cu at (150.0, 110.5)
- added G***: LOGO, Logo:Spin_Arrow, B.Cu at (150.0, 100.0)
- added R1: 130R, Resistor_SMD:R_0402_1005Metric, B.Cu at (161.0, 99.0)
- J1: moved to B.Cu
- turned J1 to -90 degrees
Connections:
- U1 pad 10: Net-(TP5-Pad1) -> unconnected-(U1-TEST-Pad10)
- U1 pad 6: Net-(TP1-Pad1) -> unconnected-(U1-TEST-Pad6)
- U1 pad 7: Net-(TP2-Pad1) -> unconnected-(U1-TEST-Pad7)
- U1 pad 8: Net-(TP3-Pad1) -> unconnected-(U1-TEST-Pad8)
- U1 pad 9: Net-(TP4-Pad1) -> unconnected-(U1-TEST-Pad9)
Routing:
- net VDD: track 28.3 -> 38.5 mm, vias 0 -> 1
- net Net-(J1-Pin_1): track 9.66 -> 13.3 mm, vias 0 -> 1
- net Net-(D1-A): track 0.00 -> 1.70 mm
- net Net-(J1-Pin_2): track 12.4 -> 14.1 mm, vias 0 -> 1
- net Net-(J1-Pin_5): track 20.2 -> 19.0 mm, vias 0 -> 1
- net Net-(J1-Pin_3): track 20.9 -> 21.7 mm, vias 0 -> 1
- net Net-(J1-Pin_4): track 17.2 -> 17.9 mm, vias 0 -> 1
Other:
- board text added: "3v3"
- board text added: "CLK"
- board text added: "CSn"
- board text added: "GND"
- board text added: "MISO"
- board text added: "MOSI"
- board text added: "PWM"
- board text added: "V1.0"
