File: MagneticSensor/MagneticSensor.kicad_sch (KiCad schematic)
At the start: 10 parts, among them J1 Conn_01x07_MountingPin, U1 AS5048A

Commit message: Initial mag encoder board
Parts:
- removed TP1, TP2, TP3, TP4, TP5: TestPoint, TestPoint:TestPoint_Pad_D1.0mm, symbol Connector:TestPoint
- added C1: 100nf, Capacitor_SMD:C_0402_1005Metric, symbol Device:C
- added C2: 10uf, Capacitor_SMD:C_0603_1608Metric, symbol Device:C
- added D1: LED, LED_SMD:LED_0603_1608Metric, symbol Device:LED
- added R1: 130R, Resistor_SMD:R_0402_1005Metric, symbol Device:R
- J1: Part (none) -> SM07B-SRSS-TB
- U1: Part (none) -> AS5048A-HTSP-500
Connections:
- net GND: now also C1.2, C2.2, D1.1 (K)
- net VDD: now also U1.11 (VDD5V), C1.1, C2.1, R1.2
- new net: D1.2 (A), R1.1
- no-connect marks 0 -> 5
