File: MotionControl.kicad_pcb (KiCad board)
At the start: 2 copper layers, 202 parts, among them J1 Screw_Terminal_01x02, J2 Conn_ARM_JTAG_SWD_10, J3 Screw_Terminal_01x04, J4 Screw_Terminal_01x02, J5 Screw_Terminal_01x04, J6 Screw_Terminal_01x04, J7 Screw_Terminal_01x04, P1 USB_C_Plug_USB2.0, Q1 2N7002, Q10 CSD18533Q5A, Q11 CSD18533Q5A, Q12 CSD18533Q5A, Q13 CSD18533Q5A, Q14 CSD18533Q5A, Q15 CSD18533Q5A, Q16 CSD18533Q5A, Q17 CSD18533Q5A, Q18 CSD18533Q5A, Q19 CSD18533Q5A, Q2 CSD18533Q5A, Q20 CSD18533Q5A, Q21 CSD18533Q5A, Q22 CSD18533Q5A, Q23 CSD18533Q5A, Q24 CSD18533Q5A, Q25 CSD18533Q5A, Q26 CSD18533Q5A, Q27 CSD18533Q5A, Q28 CSD18533Q5A, Q29 CSD18533Q5A, Q3 CSD18533Q5A, Q30 CSD18533Q5A, Q31 CSD18533Q5A, Q32 CSD18533Q5A, Q33 CSD18533Q5A, Q4 CSD18533Q5A, Q5 CSD18533Q5A, Q6 CSD18533Q5A, Q7 CSD18533Q5A, Q8 CSD18533Q5A, Q9 CSD18533Q5A, SW1 SW_Push, U1 ATSAMD21J18A-A, U2 AP2112K-3.3, U3 TMC5160A-TA, U4 TMC5160A-TA, U5 TMC5160A-TA, U6 TMC5160A-TA, Y1 32.768kHz

Commit message: Lots of work
Parts:
- removed Q10, Q11, Q12, Q13, Q18, Q19, Q20, Q21, Q22, Q23, Q24, Q25, Q26, Q27, Q28, Q29, Q30, Q31, Q32, Q33: CSD18533Q5A, Package_TO_SOT_SMD:TDSON-8-1
- added C68: 0.1uF, Capacitor_SMD:C_0402_1005Metric, F.Cu at (131.5, 117.8)
- added D11: WS2812B-2020, LED_SMD:LED_WS2812B-Mini_PLCC4_3.5x3.5mm, F.Cu at (133.3, 114.2)
- added Q34: ~, easyeda2kicad:POWERPAK-SO-8_L6.2-W5.2-P1.27-BL_POWERPAK, F.Cu at (167.3, 111.6)
- added Q35: ~, easyeda2kicad:POWERPAK-SO-8_L6.2-W5.2-P1.27-BL_POWERPAK, F.Cu at (167.3, 121.1)
- added Q36: ~, easyeda2kicad:POWERPAK-SO-8_L6.2-W5.2-P1.27-BL_POWERPAK, F.Cu at (167.3, 130.6)
- added Q37: ~, easyeda2kicad:POWERPAK-SO-8_L6.2-W5.2-P1.27-BL_POWERPAK, F.Cu at (53.2, 52.4)
- added U7: TC4427, Package_SO:SOIC-8_3.9x4.9mm_P1.27mm, F.Cu at (225.4, 106.2)
- D10, D7, D8, D9: footprint LED_SMD:LED_WS2812B-2020_PLCC4_2.0x2.0mm -> LED_SMD:LED_WS2812B-Mini_PLCC4_3.5x3.5mm
- Q14, Q15, Q16, Q17, Q2, Q3, Q4, Q5, Q6, Q7, Q8, Q9: value CSD18533Q5A -> ~; footprint Package_TO_SOT_SMD:TDSON-8-1 -> easyeda2kicad:POWERPAK-SO-8_L6.2-W5.2-P1.27-BL_POWERPAK
- R13, R16, R20, R23, R27, R30, R34, R37: footprint Resistor_SMD:R_1206_3216Metric -> Resistor_SMD:R_2512_6332Metric
- moved Q5 122.2 mm to (43.2, 39.4)
- moved Q9 118.5 mm to (53.2, 39.4)
- moved R35 112.4 mm to (131.5, 158.2)
- moved C46 92.1 mm to (120.0, 157.0)
- moved C52 92.1 mm to (124.0, 157.0)
- moved C42 92.1 mm to (120.0, 152.0)
- moved C43 92.1 mm to (120.0, 154.5)
- moved C47 92.1 mm to (120.0, 159.5)
- moved C48 92.1 mm to (120.0, 162.0)
- moved C50 92.1 mm to (124.0, 152.0)
- moved C51 92.1 mm to (124.0, 154.5)
- moved C53 92.1 mm to (124.0, 159.5)
- moved R24 92.1 mm to (124.0, 162.0)
- moved J6 87.3 mm to (102.5, 145.9)
- moved U5 86.6 mm to (103.6, 156.4)
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Connections:
- C12 pad 2: /Steppers/GND -> GND
- C14 pad 2: /Steppers/GND -> GND
- C16 pad 1: /Steppers/GND -> GND
- C17 pad 1: /Steppers/GND -> GND
- C18 pad 2: /Steppers/GND -> GND
- C20 pad 1: /Steppers/GND -> GND
- C21 pad 1: /Steppers/VLED -> +5V
- C21 pad 2: /Steppers/GND -> GND
- C24 pad 1: /Steppers/GND -> GND
- C26 pad 2: /Steppers/GND -> GND
- C28 pad 2: /Steppers/GND -> GND
- C30 pad 1: /Steppers/GND -> GND
- C31 pad 1: /Steppers/GND -> GND
- C32 pad 2: /Steppers/GND -> GND
- C34 pad 1: /Steppers/GND -> GND
- C35 pad 1: /Steppers/VLED -> +5V
- C35 pad 2: /Steppers/GND -> GND
- C38 pad 1: /Steppers/GND -> GND
- C40 pad 2: /Steppers/GND -> GND
- C42 pad 2: /Steppers/GND -> GND
- C44 pad 1: /Steppers/GND -> GND
- C45 pad 1: /Steppers/GND -> GND
- C46 pad 2: /Steppers/GND -> GND
- C48 pad 1: /Steppers/GND -> GND
- C49 pad 1: /Steppers/VLED -> +5V
- C49 pad 2: /Steppers/GND -> GND
- C52 pad 1: /Steppers/GND -> GND
- C54 pad 2: /Steppers/GND -> GND
- C56 pad 2: /Steppers/GND -> GND
- C58 pad 1: /Steppers/GND -> GND
- C59 pad 1: /Steppers/GND -> GND
- C60 pad 2: /Steppers/GND -> GND
- C62 pad 1: /Steppers/GND -> GND
- C63 pad 1: /Steppers/VLED -> +5V
- C63 pad 2: /Steppers/GND -> GND
- C66 pad 1: /Steppers/GND -> GND
- D10 pad 1: /Steppers/Stepper Unit3/LED_OUT -> +5V
- D10 pad 2: /Steppers/GND -> /Steppers/Stepper Unit3/LED_OUT
- D10 pad 3: /Steppers/Stepper Unit2/LED_OUT -> GND
- D10 pad 4: /Steppers/VLED -> /Steppers/Stepper Unit2/LED_OUT
- D7 pad 1: /Steppers/Stepper Unit/LED_OUT -> +5V
- D7 pad 2: /Steppers/GND -> /Steppers/Stepper Unit/LED_OUT
- D7 pad 3: /Steppers/Stepper Unit/LED_IN -> GND
- D7 pad 4: /Steppers/VLED -> /Steppers/Stepper Unit/LED_IN
- D8 pad 1: /Steppers/Stepper Unit1/LED_OUT -> +5V
- D8 pad 2: /Steppers/GND -> /Steppers/Stepper Unit1/LED_OUT
- D8 pad 3: /Steppers/Stepper Unit/LED_OUT -> GND
- D8 pad 4: /Steppers/VLED -> /Steppers/Stepper Unit/LED_OUT
- D9 pad 1: /Steppers/Stepper Unit2/LED_OUT -> +5V
- D9 pad 2: /Steppers/GND -> /Steppers/Stepper Unit2/LED_OUT
- D9 pad 3: /Steppers/Stepper Unit1/LED_OUT -> GND
- D9 pad 4: /Steppers/VLED -> /Steppers/Stepper Unit1/LED_OUT
- J3 pad 1: /Steppers/Stepper Unit/BMA1 -> /Steppers/Stepper Unit/BMA2
- J3 pad 2: /Steppers/Stepper Unit/BMA2 -> /Steppers/Stepper Unit/BMA1
- J3 pad 3: /Steppers/Stepper Unit/BMB1 -> /Steppers/Stepper Unit/BMB2
- J3 pad 4: /Steppers/Stepper Unit/BMB2 -> /Steppers/Stepper Unit/BMB1
- J4 pad 1: /Steppers/GND -> GND
- J5 pad 1: /Steppers/Stepper Unit1/BMA1 -> /Steppers/Stepper Unit1/BMA2
- J5 pad 2: /Steppers/Stepper Unit1/BMA2 -> /Steppers/Stepper Unit1/BMA1
- J5 pad 3: /Steppers/Stepper Unit1/BMB1 -> /Steppers/Stepper Unit1/BMB2
- J5 pad 4: /Steppers/Stepper Unit1/BMB2 -> /Steppers/Stepper Unit1/BMB1
- J6 pad 1: /Steppers/Stepper Unit2/BMA1 -> /Steppers/Stepper Unit2/BMA2
- J6 pad 2: /Steppers/Stepper Unit2/BMA2 -> /Steppers/Stepper Unit2/BMA1
- J6 pad 3: /Steppers/Stepper Unit2/BMB1 -> /Steppers/Stepper Unit2/BMB2
- J6 pad 4: /Steppers/Stepper Unit2/BMB2 -> /Steppers/Stepper Unit2/BMB1
- J7 pad 1: /Steppers/Stepper Unit3/BMA1 -> /Steppers/Stepper Unit3/BMA2
- J7 pad 2: /Steppers/Stepper Unit3/BMA2 -> /Steppers/Stepper Unit3/BMA1
- J7 pad 3: /Steppers/Stepper Unit3/BMB1 -> /Steppers/Stepper Unit3/BMB2
- J7 pad 4: /Steppers/Stepper Unit3/BMB2 -> /Steppers/Stepper Unit3/BMB1
- JP10 pad 1: /Steppers/VLOGIC -> +3V3
- JP11 pad 1: /Steppers/GND -> GND
- JP11 pad 3: /Steppers/VLOGIC -> +3V3
- JP12 pad 1: /Steppers/VLOGIC -> +3V3
- JP12 pad 3: /Steppers/GND -> GND
- JP13 pad 1: /Steppers/VLOGIC -> +3V3
- JP2 pad 1: /Steppers/VLOGIC -> +3V3
- JP3 pad 1: /Steppers/GND -> GND
- JP3 pad 3: /Steppers/VLOGIC -> +3V3
- JP4 pad 1: /Steppers/VLOGIC -> +3V3
- JP4 pad 3: /Steppers/GND -> GND
- JP5 pad 1: /Steppers/GND -> GND
- JP5 pad 3: /Steppers/VLOGIC -> +3V3
- JP6 pad 1: /Steppers/VLOGIC -> +3V3
- JP6 pad 3: /Steppers/GND -> GND
- JP7 pad 1: /Steppers/VLOGIC -> +3V3
- JP8 pad 1: /Steppers/GND -> GND
- JP8 pad 3: /Steppers/VLOGIC -> +3V3
- JP9 pad 1: /Steppers/VLOGIC -> +3V3
- JP9 pad 3: /Steppers/GND -> GND
- Q14 pad 1: /Steppers/Stepper Unit1/BMB1 -> /Steppers/Stepper Unit/HA1
- Q14 pad 2: /Steppers/Stepper Unit1/BMB1 -> /Steppers/Stepper Unit/BMA1
- Q14 pad 3: /Steppers/Stepper Unit1/BMB1 -> /Steppers/Stepper Unit/BMA2
- Q14 pad 4: /Steppers/Stepper Unit1/HB1 -> /Steppers/Stepper Unit/HA2
- Q15 pad 1: /Steppers/Stepper Unit1/SA -> /Steppers/Stepper Unit1/HA1
- Q15 pad 2: /Steppers/Stepper Unit1/SA -> /Steppers/Stepper Unit1/BMA1
- Q15 pad 3: /Steppers/Stepper Unit1/SA -> /Steppers/Stepper Unit1/BMA2
- Q15 pad 4: /Steppers/Stepper Unit1/LB1 -> /Steppers/Stepper Unit1/HA2
- Q15 pad 5: /Steppers/Stepper Unit1/BMB1 -> VM
- Q16 pad 1: /Steppers/Stepper Unit1/BMB2 -> /Steppers/Stepper Unit2/HA1
- Q16 pad 2: /Steppers/Stepper Unit1/BMB2 -> /Steppers/Stepper Unit2/BMA1
- Q16 pad 3: /Steppers/Stepper Unit1/BMB2 -> /Steppers/Stepper Unit2/BMA2
- Q16 pad 4: /Steppers/Stepper Unit1/HB2 -> /Steppers/Stepper Unit2/HA2
- Q17 pad 1: /Steppers/Stepper Unit1/SA -> /Steppers/Stepper Unit3/HA1
- Q17 pad 2: /Steppers/Stepper Unit1/SA -> /Steppers/Stepper Unit3/BMA1
- Q17 pad 3: /Steppers/Stepper Unit1/SA -> /Steppers/Stepper Unit3/BMA2
- Q17 pad 4: /Steppers/Stepper Unit1/LB2 -> /Steppers/Stepper Unit3/HA2
- Q17 pad 5: /Steppers/Stepper Unit1/BMB2 -> VM
- Q2 pad 1: /Steppers/Stepper Unit/BMA1 -> /Steppers/Stepper Unit/LA1
- Q2 pad 2: /Steppers/Stepper Unit/BMA1 -> /Steppers/Stepper Unit/SA
- Q2 pad 3: /Steppers/Stepper Unit/BMA1 -> /Steppers/Stepper Unit/SA
- Q2 pad 4: /Steppers/Stepper Unit/HA1 -> /Steppers/Stepper Unit/LA2
- Q2 pad 5: VM -> /Steppers/Stepper Unit/BMA1
- Q3 pad 1: /Steppers/Stepper Unit/SA -> /Steppers/Stepper Unit1/LA1
- Q3 pad 2: /Steppers/Stepper Unit/SA -> /Steppers/Stepper Unit1/SA
- Q3 pad 3: /Steppers/Stepper Unit/SA -> /Steppers/Stepper Unit1/SA
- Q3 pad 4: /Steppers/Stepper Unit/LA1 -> /Steppers/Stepper Unit1/LA2
- Q3 pad 5: /Steppers/Stepper Unit/BMA1 -> /Steppers/Stepper Unit1/BMA1
- Q4 pad 1: /Steppers/Stepper Unit/BMA2 -> /Steppers/Stepper Unit2/LA1
- Q4 pad 2: /Steppers/Stepper Unit/BMA2 -> /Steppers/Stepper Unit2/SA
- Q4 pad 3: /Steppers/Stepper Unit/BMA2 -> /Steppers/Stepper Unit2/SA
- Q4 pad 4: /Steppers/Stepper Unit/HA2 -> /Steppers/Stepper Unit2/LA2
- Q4 pad 5: VM -> /Steppers/Stepper Unit2/BMA1
- Q5 pad 1: /Steppers/Stepper Unit/SA -> /Steppers/Stepper Unit3/LA1
- Q5 pad 2: /Steppers/Stepper Unit/SA -> /Steppers/Stepper Unit3/SA
- Q5 pad 3: /Steppers/Stepper Unit/SA -> /Steppers/Stepper Unit3/SA
- Q5 pad 4: /Steppers/Stepper Unit/LA2 -> /Steppers/Stepper Unit3/LA2
- Q5 pad 5: /Steppers/Stepper Unit/BMA2 -> /Steppers/Stepper Unit3/BMA1
- Q6 pad 1: /Steppers/Stepper Unit/BMB1 -> /Steppers/Stepper Unit/LB1
- Q6 pad 2: /Steppers/Stepper Unit/BMB1 -> /Steppers/Stepper Unit/SB
- Q6 pad 3: /Steppers/Stepper Unit/BMB1 -> /Steppers/Stepper Unit/SB
- Q6 pad 4: /Steppers/Stepper Unit/HB1 -> /Steppers/Stepper Unit/LB2
- Q6 pad 5: VM -> /Steppers/Stepper Unit/BMB1
- Q7 pad 1: /Steppers/Stepper Unit/SA -> /Steppers/Stepper Unit1/LB1
- Q7 pad 2: /Steppers/Stepper Unit/SA -> /Steppers/Stepper Unit1/SB
- Q7 pad 3: /Steppers/Stepper Unit/SA -> /Steppers/Stepper Unit1/SB
- Q7 pad 4: /Steppers/Stepper Unit/LB1 -> /Steppers/Stepper Unit1/LB2
- Q7 pad 5: /Steppers/Stepper Unit/BMB1 -> /Steppers/Stepper Unit1/BMB1
- Q8 pad 1: /Steppers/Stepper Unit/BMB2 -> /Steppers/Stepper Unit2/LB1
- Q8 pad 2: /Steppers/Stepper Unit/BMB2 -> /Steppers/Stepper Unit2/SB
- Q8 pad 3: /Steppers/Stepper Unit/BMB2 -> /Steppers/Stepper Unit2/SB
- Q8 pad 4: /Steppers/Stepper Unit/HB2 -> /Steppers/Stepper Unit2/LB2
- Q8 pad 5: VM -> /Steppers/Stepper Unit2/BMB1
- Q9 pad 1: /Steppers/Stepper Unit/SA -> /Steppers/Stepper Unit3/LB1
- Q9 pad 2: /Steppers/Stepper Unit/SA -> /Steppers/Stepper Unit3/SB
- Q9 pad 3: /Steppers/Stepper Unit/SA -> /Steppers/Stepper Unit3/SB
- Q9 pad 4: /Steppers/Stepper Unit/LB2 -> /Steppers/Stepper Unit3/LB2
- Q9 pad 5: /Steppers/Stepper Unit/BMB2 -> /Steppers/Stepper Unit3/BMB1
- R12 pad 1: /Steppers/GND -> GND
- R13 pad 2: /Steppers/GND -> GND
- R14 pad 1: /Steppers/Stepper Unit/SA -> /Steppers/Stepper Unit/SB
- R15 pad 1: /Steppers/GND -> GND
- R16 pad 1: /Steppers/Stepper Unit/SA -> /Steppers/Stepper Unit/SB
- R16 pad 2: /Steppers/GND -> GND
- R19 pad 1: /Steppers/GND -> GND
- R20 pad 2: /Steppers/GND -> GND
- R21 pad 1: /Steppers/Stepper Unit1/SA -> /Steppers/Stepper Unit1/SB
- R22 pad 1: /Steppers/GND -> GND
- R23 pad 1: /Steppers/Stepper Unit1/SA -> /Steppers/Stepper Unit1/SB
- R23 pad 2: /Steppers/GND -> GND
- R26 pad 1: /Steppers/GND -> GND
- R27 pad 2: /Steppers/GND -> GND
- R28 pad 1: /Steppers/Stepper Unit2/SA -> /Steppers/Stepper Unit2/SB
- R29 pad 1: /Steppers/GND -> GND
- R30 pad 1: /Steppers/Stepper Unit2/SA -> /Steppers/Stepper Unit2/SB
- R30 pad 2: /Steppers/GND -> GND
- R33 pad 1: /Steppers/GND -> GND
- R34 pad 2: /Steppers/GND -> GND
- R35 pad 1: /Steppers/Stepper Unit3/SA -> /Steppers/Stepper Unit3/SB
- R36 pad 1: /Steppers/GND -> GND
- R37 pad 1: /Steppers/Stepper Unit3/SA -> /Steppers/Stepper Unit3/SB
- R37 pad 2: /Steppers/GND -> GND
- U3 pad 11: /Steppers/GND -> GND
- U3 pad 12: /Steppers/GND -> GND
- U3 pad 19: /Steppers/GND -> GND
- U3 pad 20: /Steppers/VLOGIC -> +3V3
- U3 pad 30: /Steppers/GND -> GND
- U3 pad 49: /Steppers/GND -> GND
- U3 pad 6: /Steppers/GND -> GND
- U4 pad 11: /Steppers/GND -> GND
- U4 pad 12: /Steppers/GND -> GND
- U4 pad 19: /Steppers/GND -> GND
- U4 pad 20: /Steppers/VLOGIC -> +3V3
- U4 pad 30: /Steppers/GND -> GND
- U4 pad 49: /Steppers/GND -> GND
- U4 pad 6: /Steppers/GND -> GND
- U5 pad 11: /Steppers/GND -> GND
- U5 pad 12: /Steppers/GND -> GND
- U5 pad 19: /Steppers/GND -> GND
- U5 pad 20: /Steppers/VLOGIC -> +3V3
- U5 pad 30: /Steppers/GND -> GND
- U5 pad 49: /Steppers/GND -> GND
- U5 pad 6: /Steppers/GND -> GND
- U6 pad 11: /Steppers/GND -> GND
- U6 pad 12: /Steppers/GND -> GND
- U6 pad 19: /Steppers/GND -> GND
- U6 pad 20: /Steppers/VLOGIC -> +3V3
- U6 pad 30: /Steppers/GND -> GND
- U6 pad 49: /Steppers/GND -> GND
- U6 pad 6: /Steppers/GND -> GND
Routing:
- net /Steppers/Stepper Unit3/LB1: track 0.00 -> 36.9 mm, vias 0 -> 2
- net /Steppers/Stepper Unit3/LB2: track 0.00 -> 35.2 mm, vias 0 -> 2
- net /Steppers/Stepper Unit3/HB1: track 0.00 -> 33.4 mm, vias 0 -> 2
- net /Steppers/Stepper Unit3/BMB2: track 0.00 -> 31.4 mm, vias 0 -> 2
- net /Steppers/Stepper Unit3/HA1: track 0.00 -> 30.4 mm
- net /Steppers/Stepper Unit3/HB2: track 0.00 -> 29.6 mm, vias 0 -> 2
- net /Steppers/Stepper Unit3/BMB1: track 0.00 -> 23.8 mm, vias 0 -> 2
- net +5V: track 0.00 -> 2.87 mm
- net /Steppers/Stepper Unit3/CB2: track 0.00 -> 2.29 mm
- net /Steppers/Stepper Unit3/BMA1: track 0.00 -> 2.28 mm
- net /Steppers/Stepper Unit3/SA: track 0.00 -> 1.27 mm
- added copper zone on B.Cu, net /Steppers/Stepper Unit3/BMA1
- added copper zone on F.Cu, net /Steppers/Stepper Unit3/BMA1
- added copper zone on B.Cu, net /Steppers/Stepper Unit3/BMA2
- added copper zone on F.Cu, net /Steppers/Stepper Unit3/BMA2
- added copper zone on B.Cu, net /Steppers/Stepper Unit3/BMB1
- added copper zone on F.Cu, net /Steppers/Stepper Unit3/BMB1
- added copper zone on B.Cu, net /Steppers/Stepper Unit3/BMB2
- added copper zone on F.Cu, net /Steppers/Stepper Unit3/BMB2
- added copper zone on B.Cu, net /Steppers/Stepper Unit3/SA
- added copper zone on F.Cu, net /Steppers/Stepper Unit3/SA
- added copper zone on B.Cu, net /Steppers/Stepper Unit3/SB
- added copper zone on F.Cu, net /Steppers/Stepper Unit3/SB
- added copper zone on B.Cu, net GND
- added copper zone on F.Cu, net GND
- added copper zone on F.Cu, net VM
Other:
- board outline added: 170 x 80 mm

Commit message: first stepper unit
Parts:
- removed J4: Screw_Terminal_01x02, Connector_Phoenix_SPT:PhoenixContact_SPT_5_2-H-7.5-ZB_1x02_P7.5mm_Horizontal
- removed JP11, JP12, JP3, JP4, JP5, JP6, JP8, JP9: SolderJumper_3_Bridged12, Jumper:SolderJumper-3_P1.3mm_Bridged12_RoundedPad1.0x1.5mm
- removed Q34, Q35, Q36, Q37: ~, easyeda2kicad:POWERPAK-SO-8_L6.2-W5.2-P1.27-BL_POWERPAK
- removed TP1, TP10, TP11, TP12, TP13, TP14, TP15, TP16, TP17, TP18, TP19, TP2, TP20, TP21, TP22, TP23, TP24, TP3, TP4, TP5, TP6, TP7, TP8, TP9: TestPoint, TestPoint:TestPoint_Pad_D1.5mm
- added J10: Screw_Terminal_01x02, Connector_Phoenix_MSTB:PhoenixContact_MSTBVA_2,5_2-G-5,08_1x02_P5.08mm_Vertical, F.Cu at (69.8, 28.7)
- added J11: Screw_Terminal_01x02, Connector_Phoenix_MSTB:PhoenixContact_MSTBVA_2,5_2-G-5,08_1x02_P5.08mm_Vertical, F.Cu at (243.2, 81.4)
- added J8: Screw_Terminal_01x02, Connector_Phoenix_MSTB:PhoenixContact_MSTBVA_2,5_2-G-5,08_1x02_P5.08mm_Vertical, F.Cu at (243.2, 59.2)
- added J9: Screw_Terminal_01x02, Connector_Phoenix_MSTB:PhoenixContact_MSTBVA_2,5_2-G-5,08_1x02_P5.08mm_Vertical, F.Cu at (243.2, 70.3)
- added Q10: Q_NMOS_DGS, FET:Diodes_DMT6016LFDF, F.Cu at (219.7, 46.3)
- added Q11: Q_NMOS_DGS, FET:Diodes_DMT6016LFDF, F.Cu at (219.7, 80.6)
- added Q12: Q_NMOS_DGS, FET:Diodes_DMT6016LFDF, F.Cu at (252.1, 31.7)
- added Q13: Q_NMOS_DGS, FET:Diodes_DMT6016LFDF, F.Cu at (38.4, 40.0)
- added Q18: Q_NMOS_DGS, FET:Diodes_DMT6016LFDF, F.Cu at (252.1, 39.0)
- added Q19: Q_NMOS_DGS, FET:Diodes_DMT6016LFDF, F.Cu at (252.1, 42.7)
- added Q20: Q_NMOS_DGS, FET:Diodes_DMT6016LFDF, F.Cu at (45.1, 40.0)
- added Q21: Q_NMOS_DGS, FET:Diodes_DMT6016LFDF, F.Cu at (41.5, 40.0)
- added Q22: Q_NMOS_DGS, FET:Diodes_DMT6016LFDF, F.Cu at (252.1, 46.3)
- added Q23: Q_NMOS_DGS, FET:Diodes_DMT6016LFDF, F.Cu at (256.3, 31.7)
- added Q24: Q_NMOS_DGS, FET:Diodes_DMT6016LFDF, F.Cu at (61.5, 40.0)
- added Q25: Q_NMOS_DGS, FET:Diodes_DMT6016LFDF, F.Cu at (51.8, 40.0)
- added Q26: Q_NMOS_DGS, FET:Diodes_DMT6016LFDF, F.Cu at (223.9, 35.4)
- added Q27: Q_NMOS_DGS, FET:Diodes_DMT6016LFDF, F.Cu at (223.9, 39.0)
- added Q28: Q_NMOS_DGS, FET:Diodes_DMT6016LFDF, F.Cu at (223.9, 69.6)
- added Q29: Q_NMOS_DGS, FET:Diodes_DMT6016LFDF, F.Cu at (223.9, 73.2)
- added Q30: Q_NMOS_DGS, FET:Diodes_DMT6016LFDF, F.Cu at (256.3, 35.4)
- added Q31: Q_NMOS_DGS, FET:Diodes_DMT6016LFDF, F.Cu at (256.3, 39.0)
- added Q32: Q_NMOS_DGS, FET:Diodes_DMT6016LFDF, F.Cu at (58.4, 40.0)
- added Q33: Q_NMOS_DGS, FET:Diodes_DMT6016LFDF, F.Cu at (54.8, 40.0)
- Q14, Q15, Q16, Q17, Q2, Q3, Q4, Q5, Q6, Q7, Q8, Q9: value ~ -> Q_NMOS_DGS; footprint easyeda2kicad:POWERPAK-SO-8_L6.2-W5.2-P1.27-BL_POWERPAK -> FET:Diodes_DMT6016LFDF
- moved JP10 201.6 mm to (266.8, 44.2)
- moved C40 197.1 mm to (260.4, 49.0)
- moved D9 190.1 mm to (261.4, 44.9)
- moved R25 185.5 mm to (264.4, 19.7)
- moved R26 185.5 mm to (264.4, 21.7)
- moved R29 185.5 mm to (264.4, 25.7)
- moved C41 185.5 mm to (267.3, 19.7)
- moved C44 185.5 mm to (267.3, 21.7)
- moved C45 185.5 mm to (267.3, 23.7)
- moved C49 185.5 mm to (267.3, 25.6)
- moved J6 185.5 mm to (243.2, 25.0)
- moved R28 185.5 mm to (264.4, 23.7)
- moved U5 185.5 mm to (244.3, 35.5)
- moved C42 185.2 mm to (260.2, 31.1)
- moved C43 185.2 mm to (260.2, 33.6)
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Connections:
- C12 pad 1: VM -> /Steppers/Stepper Unit/VMOT
- C14 pad 1: VM -> /Steppers/Stepper Unit/VMOT
- C15 pad 1: VM -> /Steppers/Stepper Unit/VMOT
- C20 pad 2: VM -> /Steppers/Stepper Unit/VMOT
- C24 pad 2: VM -> /Steppers/Stepper Unit/VMOT
- C26 pad 1: VM -> /Steppers/Stepper Unit1/VMOT
- C28 pad 1: VM -> /Steppers/Stepper Unit1/VMOT
- C29 pad 1: VM -> /Steppers/Stepper Unit1/VMOT
- C34 pad 2: VM -> /Steppers/Stepper Unit1/VMOT
- C38 pad 2: VM -> /Steppers/Stepper Unit1/VMOT
- C40 pad 1: VM -> /Steppers/Stepper Unit2/VMOT
- C42 pad 1: VM -> /Steppers/Stepper Unit2/VMOT
- C43 pad 1: VM -> /Steppers/Stepper Unit2/VMOT
- C48 pad 2: VM -> /Steppers/Stepper Unit2/VMOT
- C52 pad 2: VM -> /Steppers/Stepper Unit2/VMOT
- C54 pad 1: VM -> /Steppers/Stepper Unit3/VMOT
- C56 pad 1: VM -> /Steppers/Stepper Unit3/VMOT
- C57 pad 1: VM -> /Steppers/Stepper Unit3/VMOT
- C62 pad 2: VM -> /Steppers/Stepper Unit3/VMOT
- C66 pad 2: VM -> /Steppers/Stepper Unit3/VMOT
- Q14 pad 1: /Steppers/Stepper Unit/HA1 -> /Steppers/Stepper Unit/VMOT
- Q14 pad 2: /Steppers/Stepper Unit/BMA1 -> /Steppers/Stepper Unit/HA1
- Q14 pad 3: /Steppers/Stepper Unit/BMA2 -> /Steppers/Stepper Unit/BMA1
- Q15 pad 1: /Steppers/Stepper Unit1/HA1 -> /Steppers/Stepper Unit1/VMOT
- Q15 pad 2: /Steppers/Stepper Unit1/BMA1 -> /Steppers/Stepper Unit1/HA1
- Q15 pad 3: /Steppers/Stepper Unit1/BMA2 -> /Steppers/Stepper Unit1/BMA1
- Q16 pad 1: /Steppers/Stepper Unit2/HA1 -> /Steppers/Stepper Unit2/VMOT
- Q16 pad 2: /Steppers/Stepper Unit2/BMA1 -> /Steppers/Stepper Unit2/HA1
- Q16 pad 3: /Steppers/Stepper Unit2/BMA2 -> /Steppers/Stepper Unit2/BMA1
- Q17 pad 1: /Steppers/Stepper Unit3/HA1 -> /Steppers/Stepper Unit3/VMOT
- Q17 pad 2: /Steppers/Stepper Unit3/BMA1 -> /Steppers/Stepper Unit3/HA1
- Q17 pad 3: /Steppers/Stepper Unit3/BMA2 -> /Steppers/Stepper Unit3/BMA1
- Q2 pad 1: /Steppers/Stepper Unit/LA1 -> /Steppers/Stepper Unit/BMA1
- Q2 pad 2: /Steppers/Stepper Unit/SA -> /Steppers/Stepper Unit/LA1
- Q3 pad 1: /Steppers/Stepper Unit1/LA1 -> /Steppers/Stepper Unit/BMA2
- Q3 pad 2: /Steppers/Stepper Unit1/SA -> /Steppers/Stepper Unit/LA2
- Q3 pad 3: /Steppers/Stepper Unit1/SA -> /Steppers/Stepper Unit/SA
- Q4 pad 1: /Steppers/Stepper Unit2/LA1 -> /Steppers/Stepper Unit1/BMA1
- Q4 pad 2: /Steppers/Stepper Unit2/SA -> /Steppers/Stepper Unit1/LA1
- Q4 pad 3: /Steppers/Stepper Unit2/SA -> /Steppers/Stepper Unit1/SA
- Q5 pad 1: /Steppers/Stepper Unit3/LA1 -> /Steppers/Stepper Unit1/BMA2
- Q5 pad 2: /Steppers/Stepper Unit3/SA -> /Steppers/Stepper Unit1/LA2
- Q5 pad 3: /Steppers/Stepper Unit3/SA -> /Steppers/Stepper Unit1/SA
- Q6 pad 1: /Steppers/Stepper Unit/LB1 -> /Steppers/Stepper Unit/VMOT
- Q6 pad 2: /Steppers/Stepper Unit/SB -> /Steppers/Stepper Unit/HB1
- Q6 pad 3: /Steppers/Stepper Unit/SB -> /Steppers/Stepper Unit/BMB1
- Q7 pad 1: /Steppers/Stepper Unit1/LB1 -> /Steppers/Stepper Unit/VMOT
- Q7 pad 2: /Steppers/Stepper Unit1/SB -> /Steppers/Stepper Unit/HB2
- Q7 pad 3: /Steppers/Stepper Unit1/SB -> /Steppers/Stepper Unit/BMB2
- Q8 pad 1: /Steppers/Stepper Unit2/LB1 -> /Steppers/Stepper Unit1/VMOT
- Q8 pad 2: /Steppers/Stepper Unit2/SB -> /Steppers/Stepper Unit1/HB1
- Q8 pad 3: /Steppers/Stepper Unit2/SB -> /Steppers/Stepper Unit1/BMB1
- Q9 pad 1: /Steppers/Stepper Unit3/LB1 -> /Steppers/Stepper Unit1/VMOT
- Q9 pad 2: /Steppers/Stepper Unit3/SB -> /Steppers/Stepper Unit1/HB2
- Q9 pad 3: /Steppers/Stepper Unit3/SB -> /Steppers/Stepper Unit1/BMB2
- U3 pad 21: /Steppers/Stepper Unit/SD -> GND
- U3 pad 22: /Steppers/Stepper Unit/SPI -> +3V3
- U3 pad 33: VM -> /Steppers/Stepper Unit/VMOT
- U3 pad 4: VM -> /Steppers/Stepper Unit/VMOT
- U4 pad 21: /Steppers/Stepper Unit1/SD -> GND
- U4 pad 22: /Steppers/Stepper Unit1/SPI -> +3V3
- U4 pad 33: VM -> /Steppers/Stepper Unit1/VMOT
- U4 pad 4: VM -> /Steppers/Stepper Unit1/VMOT
- U5 pad 21: /Steppers/Stepper Unit2/SD -> GND
- U5 pad 22: /Steppers/Stepper Unit2/SPI -> +3V3
- U5 pad 33: VM -> /Steppers/Stepper Unit2/VMOT
- U5 pad 4: VM -> /Steppers/Stepper Unit2/VMOT
- U6 pad 21: /Steppers/Stepper Unit3/SD -> GND
- U6 pad 22: /Steppers/Stepper Unit3/SPI -> +3V3
- U6 pad 33: VM -> /Steppers/Stepper Unit3/VMOT
- U6 pad 4: VM -> /Steppers/Stepper Unit3/VMOT
Routing:
- net /Steppers/Stepper Unit3/BMB1: track 23.8 -> 86.2 mm
- net /Steppers/Stepper Unit3/BMA2: track 0.00 -> 55.4 mm, vias 0 -> 3
- net /Steppers/Stepper Unit3/BMA1: track 2.28 -> 56.9 mm, vias 0 -> 2
- net /Steppers/Stepper Unit3/HB1: track 33.4 -> 81.9 mm
- net /Steppers/Stepper Unit3/LA1: track 0.00 -> 45.7 mm, vias 0 -> 2
- net /Steppers/Stepper Unit3/SRAH: track 0.00 -> 42.0 mm, vias 0 -> 2
- net /Steppers/Stepper Unit3/BMB2: track 31.4 -> 73.0 mm
- net /Steppers/Stepper Unit3/LB1: track 36.9 -> 75.2 mm
- net /Steppers/Stepper Unit3/LB2: track 35.2 -> 68.6 mm
- net /Steppers/Stepper Unit3/HA2: track 0.00 -> 32.8 mm, vias 0 -> 2
- net /Steppers/Stepper Unit3/VMOT: track 0.00 -> 31.5 mm
- net /Steppers/Stepper Unit3/LA2: track 0.00 -> 30.5 mm, vias 0 -> 2
- net /Steppers/Stepper Unit3/HB2: track 29.6 -> 58.3 mm
- net /Steppers/Stepper Unit3/SRBH: track 0.00 -> 26.1 mm, vias 0 -> 2
- net Net-(U6-5VOUT): track 0.00 -> 16.9 mm, vias 0 -> 2
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- added copper zone on F.Cu, net /Steppers/Stepper Unit3/VMOT
- removed copper zone on B.Cu, net /Steppers/Stepper Unit3/BMA1
- removed copper zone on B.Cu, net /Steppers/Stepper Unit3/BMA2
- removed copper zone on B.Cu, net /Steppers/Stepper Unit3/BMB1
- removed copper zone on B.Cu, net /Steppers/Stepper Unit3/BMB2
- removed copper zone on B.Cu, net /Steppers/Stepper Unit3/SA
- removed copper zone on B.Cu, net /Steppers/Stepper Unit3/SB
- removed copper zone on F.Cu, net VM

Commit message: stepper unit 2 and 3, begin work on unit 4
Parts:
- U3, U4, U5, U6: footprint Package_QFP:TQFP-48-1EP_7x7mm_P0.5mm_EP5x5mm_ThermalVias -> QFP_Thermal:TQFP-48-1EP_7x7mm_P0.5mm_EP5x5mm_ThermalVias_0.3
- moved C41 180.8 mm to (91.1, 60.0), turned to -135 degrees
- moved R25 180.1 mm to (86.0, 44.2), turned to -90 degrees
- moved C44 179.0 mm to (92.2, 58.5), turned to -45 degrees
- moved C50 178.6 mm to (88.4, 62.5), turned to -135 degrees
- moved C53 176.6 mm to (90.6, 70.6), turned to -45 degrees
- moved C47 175.2 mm to (87.6, 68.5), turned to -45 degrees
- moved C45 174.2 mm to (99.4, 69.9), turned to 135 degrees
- moved C43 173.8 mm to (88.4, 60.0), turned to -135 degrees
- moved C51 173.0 mm to (95.8, 72.8)
- moved R24 169.8 mm to (95.3, 58.2)
- moved Q12 169.4 mm to (82.9, 40.0), turned to 180 degrees
- moved R26 169.3 mm to (102.2, 70.1), turned to 135 degrees
- moved C42 168.5 mm to (97.7, 75.3), turned to -45 degrees
- moved C52 168.3 mm to (99.9, 72.5), turned to 135 degrees
- moved R29 167.2 mm to (103.0, 69.3), turned to 135 degrees
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Routing:
- net (no net): track 0.00 -> 712.1 mm, vias 0 -> 49
- net +5V: track 2.87 -> 109.9 mm
- net /Steppers/Stepper Unit2/BMB1: track 0.00 -> 86.2 mm, vias 0 -> 2
- net /Steppers/Stepper Unit1/BMB1: track 0.00 -> 86.1 mm, vias 0 -> 2
- net /Steppers/Stepper Unit/BMB1: track 0.00 -> 86.1 mm
- net /Steppers/Stepper Unit2/HB1: track 0.00 -> 81.9 mm, vias 0 -> 2
- net /Steppers/Stepper Unit1/HB1: track 0.00 -> 81.8 mm, vias 0 -> 2
- net /Steppers/Stepper Unit2/LB1: track 0.00 -> 75.1 mm, vias 0 -> 2
- net /Steppers/Stepper Unit1/LB1: track 0.00 -> 75.1 mm, vias 0 -> 2
- net /Steppers/Stepper Unit2/BMB2: track 0.00 -> 72.9 mm, vias 0 -> 2
- net /Steppers/Stepper Unit1/BMB2: track 0.00 -> 72.8 mm, vias 0 -> 2
- net /Steppers/Stepper Unit/BMB2: track 0.00 -> 72.8 mm
- net /Steppers/Stepper Unit2/LB2: track 0.00 -> 71.2 mm, vias 0 -> 2
- net /Steppers/Stepper Unit1/LB2: track 0.00 -> 71.2 mm, vias 0 -> 2
- net /Steppers/Stepper Unit2/HB2: track 0.00 -> 62.8 mm, vias 0 -> 2
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- added copper zone on F.Cu, net /Steppers/Stepper Unit/BMA1
- added copper zone on F.Cu, net /Steppers/Stepper Unit/BMA2
- added copper zone on F.Cu, net /Steppers/Stepper Unit/BMB1
- added copper zone on F.Cu, net /Steppers/Stepper Unit/BMB2
- added copper zone on F.Cu, net /Steppers/Stepper Unit/SA
- added copper zone on F.Cu, net /Steppers/Stepper Unit/SB
- added copper zone on F.Cu, net /Steppers/Stepper Unit/VMOT
- added copper zone on F.Cu, net /Steppers/Stepper Unit1/BMA1
- added copper zone on F.Cu, net /Steppers/Stepper Unit1/BMA2
- added copper zone on F.Cu, net /Steppers/Stepper Unit1/BMB1
- added copper zone on F.Cu, net /Steppers/Stepper Unit1/BMB2
- added copper zone on F.Cu, net /Steppers/Stepper Unit1/SA
- added copper zone on F.Cu, net /Steppers/Stepper Unit1/SB
- added copper zone on F.Cu, net /Steppers/Stepper Unit1/VMOT
- added copper zone on F.Cu, net /Steppers/Stepper Unit2/BMA1
- added copper zone on F.Cu, net /Steppers/Stepper Unit2/BMA2
- added copper zone on F.Cu, net /Steppers/Stepper Unit2/BMB1
- added copper zone on F.Cu, net /Steppers/Stepper Unit2/BMB2
- added copper zone on F.Cu, net /Steppers/Stepper Unit2/SA
- added copper zone on F.Cu, net /Steppers/Stepper Unit2/SB
- added copper zone on F.Cu, net /Steppers/Stepper Unit2/VMOT
Other:
- board size 170 x 80 mm -> 190 x 80 mm

Commit message: Add stepper unit 4
Parts:
- moved C13 68.0 mm to (180.1, 60.0), turned to -135 degrees
- moved U3 66.5 mm to (184.4, 65.0), turned to 135 degrees
- moved C17 65.8 mm to (188.2, 70.0), turned to 180 degrees
- moved C16 65.2 mm to (181.1, 58.4), turned to -45 degrees
- moved R12 63.2 mm to (191.3, 70.0), turned to 135 degrees
- moved C22 62.8 mm to (177.3, 62.3), turned to -135 degrees
- moved R11 62.1 mm to (175.0, 44.3), turned to -90 degrees
- moved C25 61.4 mm to (179.5, 70.6), turned to -45 degrees
- moved C23 61.3 mm to (184.7, 72.7)
- moved C14 60.5 mm to (186.6, 75.4), turned to -45 degrees
- moved C19 59.4 mm to (176.6, 68.7), turned to -45 degrees
- moved R15 59.0 mm to (192.1, 69.1), turned to 135 degrees
- moved C15 57.0 mm to (177.3, 60.0), turned to -135 degrees
- moved C24 56.3 mm to (188.8, 72.4), turned to 135 degrees
- moved C18 55.1 mm to (187.8, 74.0), turned to -45 degrees
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Routing:
- net (no net): track 712.1 -> 0.00 mm, vias 49 -> 0
- net /Steppers/Stepper Unit/HB1: track 0.00 -> 81.8 mm, vias 0 -> 2
- net /Steppers/Stepper Unit/LB1: track 0.00 -> 75.1 mm, vias 0 -> 2
- net /Steppers/Stepper Unit/LB2: track 0.00 -> 71.2 mm, vias 0 -> 2
- net /Steppers/Stepper Unit/HB2: track 0.00 -> 62.7 mm, vias 0 -> 2
- net +5V: track 109.9 -> 164.2 mm
- net /Steppers/Stepper Unit/LED_OUT: track 0.00 -> 49.5 mm
- net /Steppers/Stepper Unit/BMA1: track 8.25 -> 57.2 mm, vias 0 -> 2
- net /Steppers/Stepper Unit/BMA2: track 8.79 -> 55.4 mm, vias 0 -> 3
- net /Steppers/Stepper Unit/LA1: track 0.00 -> 45.7 mm, vias 0 -> 2
- net /Steppers/Stepper Unit/SRAH: track 0.00 -> 43.6 mm, vias 0 -> 2
- net /Steppers/Stepper Unit/HA1: track 0.00 -> 32.8 mm, vias 0 -> 2
- net /Steppers/Stepper Unit/VMOT: track 0.00 -> 31.7 mm
- net /Steppers/Stepper Unit/LA2: track 0.00 -> 30.4 mm, vias 0 -> 2
- net /Steppers/Stepper Unit/HA2: track 0.00 -> 29.0 mm, vias 0 -> 2
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
Commit message: lots of changes for mcu
more routed connections
Parts:
- moved J2 145.3 mm to (100.6, 90.1)
- moved Q1 130.6 mm to (120.9, 94.8)
- moved D4 122.1 mm to (124.4, 95.0), turned to 90 degrees
- moved R5 120.7 mm to (120.5, 92.3), turned to 180 degrees
- moved R2 117.5 mm to (124.4, 92.3), turned to 90 degrees
- moved D11 115.2 mm to (134.8, 89.3)
- moved U7 113.5 mm to (142.1, 91.6), turned to 180 degrees
- moved C68 107.1 mm to (131.0, 89.4), turned to -90 degrees
- moved D5 105.2 mm to (137.4, 80.4)
- moved R8 104.4 mm to (134.7, 83.3)
- moved FB1 102.0 mm to (147.7, 89.5)
- moved R9 91.5 mm to (146.9, 80.3)
- moved D6 89.3 mm to (153.2, 81.0)
- moved C10 89.2 mm to (154.8, 97.8), turned to -90 degrees
- moved C5 89.0 mm to (143.8, 86.4)
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Connections:
- Q1 pad 1: PA17_LED -> PA16_LED
- R5 pad 2: PA17_LED -> PA16_LED
- U1 pad 15: unconnected-(U1-PA06-Pad15) -> PA06_NEOPIX
- U1 pad 35: unconnected-(U1-PA16-Pad35) -> PA16_LED
- U1 pad 36: PA17_LED -> unconnected-(U1-PA17-Pad36)
- U7 pad 2: unconnected-(U7-INA-Pad2) -> PA06_NEOPIX
Routing:
- net +3V3: track 24.4 -> 302.7 mm
- net +5V: track 164.2 -> 266.2 mm, vias 0 -> 1
- net PA16_LED: track 0.00 -> 46.1 mm
- net Net-(JP1-A): track 0.00 -> 21.2 mm
- net /D+: track 0.00 -> 20.2 mm
- net /D-: track 0.00 -> 19.5 mm, vias 0 -> 2
- net /RESETn: track 0.00 -> 16.0 mm
- net VBUS: track 0.00 -> 11.4 mm
- net Net-(U1-PA00): track 0.00 -> 7.49 mm
- net Net-(U1-PA01): track 0.00 -> 6.73 mm
- net PA06_NEOPIX: track 0.00 -> 6.64 mm
- net Net-(D11-DIN): track 0.00 -> 5.66 mm
- net Net-(U1-VDDANA): track 0.00 -> 4.08 mm
- net Net-(F1-Pad1): track 0.00 -> 3.73 mm
- net Net-(D4-K): track 0.00 -> 2.96 mm
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Other:
- board size 190 x 80 mm -> 180 x 80 mm
- board text added: "LED"
- board text added: "PWR"
- board text added: "USB"
