File: power_usb.kicad_sch (KiCad schematic)
At the start: 15 parts, among them J1 Screw_Terminal_01x02, P1 USB_C_Plug_USB2.0, U2 AP2112K-3.3

Commit message: Updated footprints, digikey parts
Parts:
- F1: Part 0ZCG0050FF2C -> PTS12066V050
- J1: Part (none) -> 1757242
Changed lines of the file:
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@@
+			)
+		)
+		(property "Part" "1757242"
+			(at 128.27 71.12 0)
+			(effects
+				(font
+					(size 1.27 1.27)
+				)
+				(hide yes)
 			)
 		)
@@
 			)
 		)
-		(property "Part" "0ZCG0050FF2C"
+		(property "Part" "PTS12066V050"
 			(at 119.38 88.9 90)
 			(effects
