File: opticalins.kicad_sch (KiCad schematic)
At the start: 12 parts, among them J16 Conn_01x03_MountingPin, J17 Conn_01x03_MountingPin, J18 Conn_01x03_MountingPin, J19 Conn_01x03_MountingPin, J20 Conn_01x03_MountingPin, J21 Conn_01x03_MountingPin, J22 Conn_01x03_MountingPin, J23 Conn_01x03_MountingPin, J24 Conn_01x03_MountingPin, J25 Conn_01x03_MountingPin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

Commit message: add spi cs pin, remove center endstop support
Parts:
- removed J18, J21, J24, J27: Conn_01x03_MountingPin, Connector_JST:JST_SH_BM03B-SRSS-TB_1x03-1MP_P1.00mm_Vertical, symbol Connector_Generic_MountingPin:Conn_01x03_MountingPin
Connections:
- net OUT10 is gone; now on net OUT7: J25.3 (Pin_3)
- net OUT11 is gone; now on net OUT8: J26.3 (Pin_3)
- net OUT3: now also J19.3 (Pin_3)
- net OUT4: now also J20.3 (Pin_3); no longer J19.3 (Pin_3)
- net OUT5: now also J22.3 (Pin_3); no longer J20.3 (Pin_3)
- net OUT6: now also J23.3 (Pin_3)
- net OUT7: no longer J22.3 (Pin_3)
- net OUT8: no longer J23.3 (Pin_3)
